File: Hardware_electronics/PCB_ADS1115/ProPrj_SKANSEN Metal Detector_2026-10-08.kicad_sch (KiCad schematic)
At the start: 15 parts, among them P1 MPF Header-Male-2.54_2x20, U1 ADS1115IDGST, U2 MCP622T-E/MF, U3 BOB-12009

Commit message: Update hardware electronics PCB and KiCad files
Parts:
- removed ?: (no value), ProPrj_SKA-easyedapro:, symbol ProPrj_SKA-easyedapro:Drawing-Symbol_A4
- removed H2: PZ254V-11-02P, ProPrj_SKA-easyedapro:HDR-TH_2P-P2.54-V-M, symbol ProPrj_SKA-easyedapro:PZ254V-11-02P
- removed R2: 10kΩ, ProPrj_SKA-easyedapro:R1206, symbol ProPrj_SKA-easyedapro:Res
- added H7: PZ254V-11-02P, JLCPCB_lib:HDR-TH_2P-P2.54-V-M, symbol ProPrj_SKA-easyedapro:PZ254V-11-02P
- added J1: Conn_01x03_Pin, Connector_PinSocket_2.54mm:PinSocket_1x03_P2.54mm_Vertical, symbol Connector:Conn_01x03_Pin
- C1: value BIPOLAR CAPACITOR 47,0 UF -> BIPOLAR CAPACITOR 100nF; footprint ProPrj_SKA-easyedapro:CAP-TH_BD13.0-P5.00-D0.6-FD -> JLCPCB_lib:CAP-TH_BD13.0-P5.00-D0.6-FD; Manufacturer Part 100nF -> BIPOLAR CAPACITOR 47,0 UF
- C2: footprint ProPrj_SKA-easyedapro:C0603 -> JLCPCB_lib:C0805
- H1: renamed from H5; footprint ProPrj_SKA-easyedapro:HDR-TH_2P-P2.54-V-M -> JLCPCB_lib:HDR-TH_2P-P2.54-V-M; Manufacturer Part 5V_CONN -> PZ254V-11-02P
- H2: renamed from H6; footprint ProPrj_SKA-easyedapro:HDR-TH_2P-P2.54-V-M -> JLCPCB_lib:HDR-TH_2P-P2.54-V-M; Manufacturer Part 3.3V_CONN -> PZ254V-11-02P
- H3: renamed from H4; footprint ProPrj_SKA-easyedapro:HDR-TH_2P-P2.54-V-M -> JLCPCB_lib:HDR-TH_2P-P2.54-V-M; Manufacturer Part GND_CONN -> PZ254V-11-02P
- H4: renamed from H3; footprint ProPrj_SKA-easyedapro:HDR-TH_2P-P2.54-V-M -> JLCPCB_lib:HDR-TH_2P-P2.54-V-M; Manufacturer Part PRESSURE_IN -> PZ254V-11-02P
- H5: renamed from H1; footprint ProPrj_SKA-easyedapro:HDR-TH_2P-P2.54-V-M -> JLCPCB_lib:HDR-TH_2P-P2.54-V-M; Manufacturer Part GPS_IN -> PZ254V-11-02P
- P1: footprint ProPrj_SKA-easyedapro:HDR-TH_40PIN-V-ROW2-COL20-FEMALE-PITCH2.54 -> JLCPCB_lib:HDR-TH_40PIN-V-ROW2-COL20-FEMALE-PITCH2.54
- R1: value 10kΩ -> 8.2k; footprint ProPrj_SKA-easyedapro:R1206 -> JLCPCB_lib:R1206
- U1: renamed from U2; footprint ProPrj_SKA-easyedapro:DFN-8_L3.0-W3.0-P0.65-BL-EP2.0 -> JLCPCB_lib:MCP622-breakout
- U2: renamed from U1; footprint ProPrj_SKA-easyedapro:VSSOP-10_L3.0-W3.0-P0.50-LS4.9-BL -> JLCPCB_lib:HDR-TH_10P-P2.54-V-F-S2.54
- U3: footprint ProPrj_SKA-easyedapro:CONV_BOB-12009 -> JLCPCB_lib:CONV_BOB-12009
Connections:
- net +5V: now also J1.1 (Pin_1)
- net GND: now also H7.2, J1.3 (Pin_3)
- net LW_IMP_SIG_2: now also U1.1 (VOUTA), U1.2 (VINA–); no longer U1.3 (VINA+)
- net Pressure Sensor Signal: now also J1.2 (Pin_2)
- new net LW_IMP_SIG_2_PREAMP: H7.1, U1.3 (VINA+)
Other:
- note removed: "Double check I did this correct"
- note removed: "PRESSURE_SENSE_1"
- moved on the sheet: H1
